Commit message: Aruco marker pose estimation FIXED.

File: src/etf_modules/sim_bringup/urdf/camera_depth_left.xacro (robot description, xacro)
@@ -1,5 +1,5 @@
 <?xml version="1.0"?>
 <robot xmlns:xacro="http://www.ros.org/wiki/xacro" name="camera_depth_left">
-	<xacro:macro name="camera_depth_left" params="camera_left_x:='1.5' camera_left_y:='-0.5' camera_left_z:='0.6' camera_left_R:='0' camera_left_P:='-0.1' camera_left_Y:='3.14159'" >
+	<xacro:macro name="camera_depth_left" params="camera_left_x:='0.85' camera_left_y:='-0.5' camera_left_z:='0.6' camera_left_R:='0' camera_left_P:='-0.1' camera_left_Y:='3.14159'" >
     <joint name="camera_joint_left" type="fixed">
         <parent link="link_base"/>

File: src/etf_modules/sim_bringup/urdf/camera_depth_right.xacro (robot description, xacro)
@@ -1,5 +1,5 @@
 <?xml version="1.0"?>
 <robot xmlns:xacro="http://www.ros.org/wiki/xacro" name="camera_depth_right">
-	<xacro:macro name="camera_depth_right" params="camera_right_x:='1.5' camera_right_y:='-0.5' camera_right_z:='0.6' camera_right_R:='0' camera_right_P:='-0.1' camera_right_Y:='3.14159'" >
+	<xacro:macro name="camera_depth_right" params="camera_right_x:='0.85' camera_right_y:='-0.5' camera_right_z:='0.6' camera_right_R:='0' camera_right_P:='-0.1' camera_right_Y:='3.14159'" >
     <joint name="camera_joint_right" type="fixed">
         <parent link="link_base"/>

File: src/etf_modules/sim_bringup/urdf/xarm_device.urdf.xacro (robot description, xacro)
@@ -28,5 +28,5 @@
   <xacro:arg name="baud_checkset" default="true"/>
   <xacro:arg name="default_gripper_baud" default="2000000"/>
-  <xacro:arg name="camera_left_x" default="1.5"/>
+  <xacro:arg name="camera_left_x" default="0.85"/>
   <xacro:arg name="camera_left_y" default="-0.5"/>
   <xacro:arg name="camera_left_z" default="0.6"/>
@@ -34,5 +34,5 @@
   <xacro:arg name="camera_left_P" default="-0.1"/>
   <xacro:arg name="camera_left_Y" default="3.14159"/>
-  <xacro:arg name="camera_right_x" default="1.5"/>
+  <xacro:arg name="camera_right_x" default="0.85"/>
   <xacro:arg name="camera_right_y" default="0.5"/>
   <xacro:arg name="camera_right_z" default="0.6"/>
